File: Hardware/Synthesizer-VHF.kicad_sch (KiCad schematic)
At the start: 81 parts, among them J1 REF Select, J2 REF_IN, J3 RFOUTA, J4 RFOUTB, J5 USB-C 2.0 16P, J7 Header 1x3, J8 Screw_Terminal_01x12, U10 ADF4350, U2 MC78L05_TO-252, U4 GM1207ACPZ-3.3, U7 GM1207ACPZ-3.3, U8 ATtiny1616-M, U9 FT231XQ, X1 IQXO-70

Commit message: Added test points for scope probes, tweaked layout a bit
Parts:
- added J6, J9: Header 1x3, Connector_PinHeader_2.54mm:PinHeader_1x03_P2.54mm_Vertical, symbol Connector:Conn_01x03_Pin
- D5: value White -> PA2
- D8: value White -> PA3
- J2, J3, J4: footprint Connector_Coaxial:SMA_Amphenol_901-143_Horizontal -> Synthesizer:SMA_Amphenol_901-143_Horizontal
Connections:
- net GND: now also J6.3 (Pin_3), J9.1 (Pin_1)
- net LD: now also J6.1 (Pin_1)
- net MUX: now also J6.2 (Pin_2)
- net at U8.10 (PB4): now also J9.3 (Pin_3)
- net at U8.9 (PB5): now also J9.2 (Pin_2)
- no-connect marks 16 -> 14
Other:
- note added: "What frequency range on output is required? all the way to 6 GHZ? What VCC/VDD pins require lowest noise? Can regulators be different noise levels on different pins to save $? On Eval Kit for ADF4350, why only two regulators? How does eval kit get away with one set or loop filter Rs and Cs? How should loop filter components be distributed between CP side and TUNE side (to minimize pickup) What co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"
- note removed: "What frequency range on output is required? all the way to 6 GHZ? Should board have 1 or 2 RF outputs? How fussy on RFOUT about trace impedance, balance, shielding? Should RFOUT use Balun or just one side to SMA? Should board use SMA or some other RF connector? Should this board be 0.032 thick or made from Rogers material? (make 50 ohm traces narrower) Should board be more than two layers? Layou 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"
- moved on the sheet: C1, C22, C24, C27, C28, C29, C6, J3, J4, R16, R17, R18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

Commit message: Tried to find a better TCXO at 40 MHz, but jlcpcb froze all of kicad several times.
Parts:
- C12: renamed from C6; LCSC (none) -> C32949
- C13: renamed from C11; LCSC (none) -> C15195
- C15: renamed from C1; LCSC (none) -> C1525
- C17: renamed from C29; LCSC (none) -> C513576
- C18: renamed from C9; LCSC (none) -> C15195
- C19: renamed from C12; LCSC (none) -> C32949
- C20: renamed from C28; LCSC (none) -> C541551
- C21: renamed from C8; LCSC (none) -> C32949
- C23: renamed from C22; LCSC (none) -> C32949
- C24: renamed from C16; LCSC (none) -> C32949
- C28: renamed from C10; LCSC (none) -> C32949
- C3: LCSC (none) -> C15195
- C30: renamed from C7; LCSC (none) -> C15195
- C31: renamed from C27; LCSC (none) -> C107121
- C4: renamed from C13; LCSC (none) -> C15195
- J5: renamed from J2; LCSC (none) -> C496551
- J7: renamed from J3; LCSC (none) -> C496551
- J9: renamed from J4; LCSC (none) -> C496551
- R11: renamed from R6; LCSC (none) -> C137960
- R14: renamed from R17; LCSC (none) -> C114536
- R15: renamed from R5; LCSC (none) -> C137960
- R2: renamed from R20; LCSC (none) -> C17168
- R20: renamed from R18; LCSC (none) -> C17477
- R21: renamed from R3; LCSC (none) -> C137960
- R23: renamed from R2; LCSC (none) -> C137960
- R25: renamed from R16; LCSC (none) -> C17513
- R5: renamed from R9; LCSC (none) -> C137960
- R6: renamed from R19; LCSC (none) -> C105876
- R7: renamed from R1; LCSC (none) -> C138052
- U4: renamed from U10; LCSC (none) -> C98705
- renumbered C26 to C1, C5 to C10, C45 to C11, C34 to C14, C2 to C16, C44 to C2, C24 to C22, C15 to C25, C4 to C26, C41 to C27, C42 to C29, C40 to C32, C35 to C33, C31 to C5, C47 to C6, C46 to C7, C48 to C8, C43 to C9, D4 to D2, D6 to D4, D7 to D5, D2 to D6, D5 to D7, J8 to J1, J6 to J2, J1 to J3, J5 to J4, J9 to J6, J7 to J8, R10 to R1, R26 to R10, R30 to R12, R25 to R13, R29 to R16, R12 to R17, R8 to R18, R28 to R19, R4 to R22, R7 to R3, R21 to R4, R27 to R8, R11 to R9, U2 to U1, U9 to U2, U8 to U3, U7 to U5, U4 to U6
Connections:
- net 12V: now also C1.1
- net at D1.1 (K), U1.3 (IN): no longer C1.1
Other:
- moved on the sheet: C1, D1
