File: Hardware/Synthesizer-VHF.kicad_pcb (KiCad board)
At the start: 4 copper layers, 38.9 x 37.7 mm, 92 parts, among them J1 Screw_Terminal_01x02, J2 Scope, J4 USB-C 2.0 16P, J5 REF_IN, J7 RFOUTA, J8 Header 1x3, J9 RFOUTB, U1 LM7805A, U2 FT231XQ, U3 ATtiny1616-M, U4 ADF435x, U5 ADP150AUJZ-3.3-R7, U6 ADP150AUJZ-3.3-R7, U7 ADP150AUJZ-3.3-R7, X1 IQXO-70

Commit message: final commit for 4 layer with parts on back side...that add a lot of cost Design uses a single supply with massive decoupling because EVKIT and Hellmich sig gen did it that way.  Also parts on back side may not improve grounding because of pwr via to get to cap.
Parts:
- C15, C43: value 120p -> 100p
Changed lines of the file:
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@@
 		)
 		(property "LCSC" "C541551"
-			(at 0 0 360)
+			(at 0 0 0)
 			(layer "F.SilkS")
 			(hide yes)
@@
 			)
 		)
+		(property "LCSC" "C29149"
+			(at 0 0 0)
+			(layer "F.SilkS")
+			(hide yes)
+			(effects
+				(font
+					(size 1.27 1.27)
+					(thickness 0.15)
+				)
+			)
+		)
 		(property ki_fp_filters "SOT?23*")
 		(sheetname "Root")
@@
 		(tags "resistor")
 		(property "Reference" "R25"
-			(at -3.1875 -0.1 360)
+			(at -3.1875 -0.1 0)
 			(layer "F.SilkS")
 			(effects
@@
 		)
 		(property "Value" "1K"
-			(at 0 1.65 360)
+			(at 0 1.65 0)
 			(layer "F.Fab")
 			(hide yes)
@@
 		)
 		(fp_text user "${REFERENCE}"
-			(at 0 0 360)
+			(at 0 0 0)
 			(layer "F.Fab")
 			(effects
@@
 		)
 		(fp_text user "${REFERENCE}"
-			(at -0.000893 0.001574 360)
+			(at -0.000893 0.001574 0)
 			(layer "F.Fab")
 			(effects
@@
 		(sheetname "Root")
 		(sheetfile "Synthesizer-VHF.kicad_sch")
-		(attr smd)
+		(attr smd exclude_from_pos_files)
 		(fp_line
 			(start -0.04 0.36)
@@
 		)
 		(fp_text user "${REFERENCE}"
-			(at -0.000893 0.001574 360)
+			(at -0.000893 0.001574 0)
 			(layer "F.Fab")
 			(effects
@@
 		)
 		(property "LCSC" "C105876"
-			(at 0 0 360)
+			(at 0 0 0)
 			(layer "F.SilkS")
 			(hide yes)
@@
 		)
 		(fp_text user "${REFERENCE}"
-			(at -0.000893 0.001574 360)
+			(at -0.000893 0.001574 0)
 			(layer "F.Fab")
 			(effects
@@
 		(tags "resistor")
 		(property "Reference" "R20"
-			(at 3.2875 -0.1 360)
+			(at 3.2875 -0.1 0)
 			(layer "F.SilkS")
 			(effects
@@
 		)
 		(property "Value" "0R"
-			(at 0 1.65 360)
+			(at 0 1.65 0)
 			(layer "F.Fab")
 			(hide yes)
@@
 		)
 		(fp_text user "${REFERENCE}"
-			(at 0 0 360)
+			(at 0 0 0)
 			(layer "F.Fab")
 			(effects
@@
 		)
 		(property "LCSC" "C144745"
-			(at 0 0 360)
+			(at 0 0 0)
 			(layer "F.SilkS")
 			(hide yes)
@@
 		(tags "capacitor")
 		(property "Reference" "C31"
-			(at 3.25 0 360)
+			(at 3.25 0 0)
 			(layer "F.SilkS")
 			(effects
@@
 		)
 		(property "Value" "680p"
-			(at 0 1.68 360)
+			(at 0 1.68 0)
 			(layer "F.Fab")
 			(hide yes)
@@
 		)
 		(fp_text user "${REFERENCE}"
-			(at 0 0 360)
+			(at 0 0 0)
 			(layer "F.Fab")
 			(effects
@@
 		)
 		(property "LCSC" "C15195"
-			(at 0 0 360)
+			(at 0 0 0)
 			(layer "F.SilkS")
 			(hide yes)
@@
 		)
 		(fp_text user "${REFERENCE}"
-			(at 0 2.54 360)
+			(at 0 2.54 0)
 			(layer "F.Fab")
 			(effects
@@
 		)
 		(property "LCSC" "C1525"
-			(at 0 0 360)
+			(at 0 0 0)
 			(layer "F.SilkS")
 			(hide yes)
@@
 		)
 		(fp_text user "${REFERENCE}"
-			(at -0.000893 0.001574 360)
+			(at -0.000893 0.001574 0)
 			(layer "F.Fab")
 			(effects
@@
 		)
 		(property "LCSC" "C15195"
-			(at 0 0 360)
+			(at 0 0 0)
 			(layer "F.SilkS")
 			(hide yes)
@@
 		)
 		(fp_text user "${REFERENCE}"
-			(at -0.000893 0.001574 360)
+			(at -0.000893 0.001574 0)
 			(layer "F.Fab")
 			(effects
@@
 		)
 		(property "LCSC" "C17168"
-			(at 0 0 360)
+			(at 0 0 0)
 			(layer "F.SilkS")
 			(hide yes)
@@
 		)
 		(fp_text user "${REFERENCE}"
-			(at 0 0 360)
+			(at 0 0 0)
 			(layer "F.Fab")
 			(effects
@@
 			)
 		)
-		(property "Value" "120p"
+		(property "Value" "100p"
 			(at 0 1.5 90)
 			(unlocked yes)
@@
 		(tags "SOT TO_SOT_SMD")
 		(property "Reference" "U6"
-			(at 0 -2.4 360)
+			(at 0 -2.4 0)
 			(layer "F.SilkS")
 			(hide yes)
@@
 		)
 		(property "Value" "ADP150AUJZ-3.3-R7"
-			(at 0 2.4 360)
+			(at 0 2.4 0)
 			(layer "F.Fab")
 			(hide yes)
@@
 		)
 		(property "Footprint" "Package_TO_SOT_SMD:SOT-23-5"
-			(at 0 0 360)
+			(at 0 0 0)
 			(layer "F.Fab")
 			(hide yes)
@@
 		)
 		(property "Datasheet" "https://www.analog.com/media/en/technical-documentation/data-sheets/adp150.pdf"
-			(at 0 0 360)
+			(at 0 0 0)
 			(layer "F.Fab")
 			(hide yes)
@@
 		)
 		(property "Description" "150mA Fixed 3.3V, 5.5V in, TSOT-23-5 Regulator"
-			(at 0 0 360)
+			(at 0 0 0)
 			(layer "F.Fab")
 			(hide yes)
@@
 			)
 		)
+		(property "LCSC" "C29149"
+			(at 0 0 0)
+			(layer "F.SilkS")
+			(hide yes)
+			(effects
+				(font
+					(size 1.27 1.27)
+					(thickness 0.15)
+				)
+			)
+		)
 		(property ki_fp_filters "SOT?23*")
 		(sheetname "Root")
@@
 		)
 		(fp_text user "${REFERENCE}"
-			(at 0 0 360)
+			(at 0 0 0)
 			(layer "F.Fab")
 			(effects
@@
 			)
 		)
-		(property "Value" "120p"
+		(property "Value" "100p"
 			(at 0 1.5 90)
 			(unlocked yes)
@@
 			)
 		)
+		(property "LCSC" "C29149"
+			(at 0 0 0)
+			(layer "F.SilkS")
+			(hide yes)
+			(effects
+				(font
+					(size 1.27 1.27)
+					(thickness 0.15)
+				)
+			)
+		)
 		(property ki_fp_filters "SOT?23*")
 		(sheetname "Root")
@@
 		)
 		(fp_text user "${REFERENCE}"
-			(at -0.000893 0.001574 360)
+			(at -0.000893 0.001574 0)
 			(layer "F.Fab")
 			(effects
@@
 		(tags "capacitor")
 		(property "Reference" "C17"
-			(at 3.25 -0.1 360)
+			(at 3.25 -0.1 0)
 			(layer "F.SilkS")
 			(effects
@@
 		)
 		(property "Value" "4.7n"
-			(at 0 1.68 360)
+			(at 0 1.68 0)
 			(layer "F.Fab")
 			(hide yes)
@@
 		)
 		(fp_text user "${REFERENCE}"
-			(at 0 0 360)
+			(at 0 0 0)
 			(layer "F.Fab")
 			(effects
@@
 		(tags "resistor")
 		(property "Reference" "R14"
-			(at -3.2 0.1 360)
+			(at -3.2 0.1 0)
 			(layer "F.SilkS")
 			(effects
@@
 		)
 		(property "Value" "560R"
-			(at 0 1.65 360)
+			(at 0 1.65 0)
 			(layer "F.Fab")
 			(hide yes)
@@
 		)
 		(fp_text user "${REFERENCE}"
-			(at 0 0 360)
+			(at 0 0 0)
 			(layer "F.Fab")
 			(effects
@@
 		)
 		(fp_text user "${REFERENCE}"
-			(at -0.000893 -0.001574 360)
+			(at -0.000893 -0.001574 0)
 			(layer "B.Fab")
 			(effects
@@
 		)
 		(fp_text user "${REFERENCE}"
-			(at -0.000893 -0.001574 360)
+			(at -0.000893 -0.001574 0)
 			(layer "B.Fab")
 			(effects
