File: hardware/Synthesizer-VHF.kicad_pcb (KiCad board)
At the start: 4 copper layers, 50.6 x 50.6 mm, 93 parts, among them J1 Screw_Terminal_01x02, J2 Scope, J4 USB-C 2.0 16P, J5 REF_IN, J6 Scope, J7 RFOUTA, J8 Header 1x3, J9 RFOUTB, U1 LM7805A, U2 FT231XQ, U3 ATtiny1616-M, U4 ADF4351, U5 USBLC6-2SC6, U7 ADP150AUJZ-3.3-R7, U8 ADP150AUJZ-3.3-R7, X1 HCI 8122S-25NQ33FTL

Commit message: diecast-2x2: User.Drawings outlines for enclosure rim (inner/outer) and 4 corner bosses + label
Other:
- board text added: "ENCLOSURE RIM / BOSS - keep pads & holes clear"
Changed lines of the file:
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@@
 		(layer "F.Mask")
+	)
+	(gr_rect
+		(start 128.75 69.55)
+		(end 136.675 77.5)
+		(stroke
+			(width 0.15)
+			(type default)
+		)
+		(fill no)
+		(layer "Dwgs.User")
+	)
+	(gr_rect
+		(start 128.75 69.55)
+		(end 179.3 120.15)
+		(stroke
+			(width 0.15)
+			(type default)
+		)
+		(fill no)
+		(layer "Dwgs.User")
+	)
+	(gr_rect
+		(start 128.75 112.2)
+		(end 136.675 120.15)
+		(stroke
+			(width 0.15)
+			(type default)
+		)
+		(fill no)
+		(layer "Dwgs.User")
+	)
+	(gr_rect
+		(start 131.175 72)
+		(end 176.875 117.7)
+		(stroke
+			(width 0.15)
+			(type default)
+		)
+		(fill no)
+		(layer "Dwgs.User")
+	)
+	(gr_rect
+		(start 171.375 69.55)
+		(end 179.3 77.5)
+		(stroke
+			(width 0.15)
+			(type default)
+		)
+		(fill no)
+		(layer "Dwgs.User")
+	)
+	(gr_rect
+		(start 171.375 112.2)
+		(end 179.3 120.15)
+		(stroke
+			(width 0.15)
+			(type default)
+		)
+		(fill no)
+		(layer "Dwgs.User")
 	)
 	(gr_arc
@@
 		)
 	)
+	(gr_text "ENCLOSURE RIM / BOSS - keep pads & holes clear"
+		(at 154.025 67.8 0)
+		(layer "Dwgs.User")
+		(effects
+			(font
+				(size 1 1)
+				(thickness 0.15)
+			)
+		)
+	)

Commit message: diecast-2x2: user layout edits (KiCad save)
Parts:
- moved J4 1.76 mm to (142.3, 76.4)
- moved J5 0.19 mm to (166.9, 76.4)
- moved J9 0.10 mm to (166.9, 113.3)
Routing:
- net /5V: track 96.7 -> 100.1 mm
- net GND: vias 204 -> 201
Changed lines of the file:
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@@
 	(footprint "Connector_Coaxial:SMA_Amphenol_901-144_Vertical"
 		(layer "B.Cu")
-		(at 167.06 76.24 180)
+		(at 166.91 76.36 180)
 		(descr "https://www.amphenolrf.com/library/download/link/link_id/593640/parent/901-144/")
 		(tags "SMA THT Female Jack Vertical")
@@
 	(footprint "Connector_Coaxial:SMA_Amphenol_901-144_Vertical"
 		(layer "B.Cu")
-		(at 166.99 113.31 180)
+		(at 166.89 113.31 180)
 		(descr "https://www.amphenolrf.com/library/download/link/link_id/593640/parent/901-144/")
 		(tags "SMA THT Female Jack Vertical")
@@
 	(footprint "Synthesizer:USB_C_Receptacle_G-Switch_GT-USB-7010ASV"
 		(layer "B.Cu")
-		(at 144.07 76.225)
+		(at 142.32 76.375)
 		(descr "USB Type C, right-angle, SMT, https://datasheet.lcsc.com/lcsc/2204071530_G-Switch-GT-USB-7010ASV_C2988369.pdf")
 		(tags "USB C Type-C Receptacle SMD")
@@
 	)
 	(via
-		(at 140.5 76.8)
-		(size 0.45)
-		(drill 0.3)
-		(layers "F.Cu" "B.Cu")
-		(capping no)
-		(covering
-			(front no)
-			(back no)
-		)
-		(plugging
-			(front no)
-			(back no)
-		)
-		(filling no)
-		(net "GND")
-	)
-	(via
 		(at 152.525 70.6375)
 		(size 0.45)
@@
 	)
 	(via
-		(at 147.6 76.8)
-		(size 0.45)
-		(drill 0.3)
-		(layers "F.Cu" "B.Cu")
-		(capping no)
-		(covering
-			(front no)
-			(back no)
-		)
-		(plugging
-			(front no)
-			(back no)
-		)
-		(filling no)
-		(net "GND")
-	)
-	(via
 		(at 149.200006 86.5)
 		(size 0.45)
@@
 	)
 	(via
-		(at 172.7 100.5)
-		(size 0.45)
-		(drill 0.3)
-		(layers "F.Cu" "B.Cu")
-		(capping no)
-		(covering
-			(front no)
-			(back no)
-		)
-		(plugging
-			(front no)
-			(back no)
-		)
-		(filling no)
-		(net "GND")
-	)
-	(via
 		(at 143.525 119.0625)
 		(size 0.45)
@@
 	)
 	(segment
-		(start 153.65408 84.7)
-		(end 153.95408 85)
-		(width 0.5)
-		(layer "F.Cu")
-		(net "/5V")
-	)
-	(segment
 		(start 170.801574 103.380893)
 		(end 169.319107 103.380893)
@@
 	)
 	(segment
+		(start 173.4 99.4)
+		(end 172.8 100)
+		(width 0.5)
+		(layer "F.Cu")
+		(net "/5V")
+	)
+	(segment
 		(start 135.441574 99.824041)
 		(end 135.717533 100.1)
@@
 	)
 	(segment
-		(start 146.8 87.070733)
-		(end 146.8 85.3)
+		(start 171.9 85)
+		(end 173.4 86.5)
 		(width 0.5)
 		(layer "F.Cu")
@@
 	)
 	(segment
-		(start 170.2 100)
-		(end 171.561574 101.361574)
-		(width 0.5)
-		(layer "F.Cu")
-		(net "/5V")
-	)
-	(segment
-		(start 146.8 85.3)
-		(end 147.4 84.7)
-		(width 0.5)
-		(layer "F.Cu")
-		(net "/5V")
-	)
-	(segment
 		(start 150.219107 87.501574)
 		(end 150.217533 87.5)
@@
 	)
 	(segment
-		(start 153.95408 85)
-		(end 171.9 85)
-		(width 0.5)
-		(layer "F.Cu")
-		(net "/5V")
-	)
-	(segment
 		(start 135.441574 99.824041)
 		(end 135.441574 93.208426)
@@
 	)
 	(segment
-		(start 171.9 85)
-		(end 172.4 85.5)
-		(width 0.5)
+		(start 151.495898 88.400202)
+		(end 151.495898 88.873426)
+		(width 0.15)
 		(layer "F.Cu")
 		(net "/5V")
 	)
 	(segment
-		(start 151.495898 88.400202)
-		(end 151.495898 88.873426)
-		(width 0.15)
+		(start 153.65408 84.7)
+		(end 153.95408 85)
+		(width 0.5)
 		(layer "F.Cu")
 		(net "/5V")
@@
 	)
 	(segment
+		(start 173.4 86.5)
+		(end 173.4 99.4)
+		(width 0.5)
+		(layer "F.Cu")
+		(net "/5V")
+	)
+	(segment
 		(start 138.378836 94)
 		(end 138.841074 94)
@@
 	)
 	(segment
+		(start 169.524999 100)
+		(end 171.561574 100)
+		(width 0.5)
+		(layer "F.Cu")
+		(net "/5V")
+	)
+	(segment
 		(start 169.3 101.5)
 		(end 169.6 101.2)
@@
 	)
 	(segment
-		(start 171.561574 101.361574)
-		(end 171.561574 103.138426)
-		(width 0.5)
+		(start 170.1375 86.2)
+		(end 170.1375 85)
+		(width 0.15)
 		(layer "F.Cu")
 		(net "/5V")
 	)
 	(segment
-		(start 170.1375 86.2)
-		(end 170.1375 85)
-		(width 0.15)
+		(start 146.8 87.070733)
+		(end 146.8 85.3)
+		(width 0.5)
 		(layer "F.Cu")
 		(net "/5V")
@@
 	)
 	(segment
+		(start 147.4 84.7)
+		(end 153.65408 84.7)
+		(width 0.5)
+		(layer "F.Cu")
+		(net "/5V")
+	)
+	(segment
 		(start 144.7 93.335)
 		(end 144.003574 93.335)
@@
 	)
 	(segment
+		(start 171.319107 103.380893)
+		(end 170.801574 103.380893)
+		(width 0.5)
+		(layer "F.Cu")
+		(net "/5V")
+	)
+	(segment
 		(start 136.6 92.315)
 		(end 137.215 92.315)
@@
 	)
 	(segment
-		(start 169.4 99.875001)
-		(end 169.524999 100)
-		(width 0.5)
-		(layer "F.Cu")
-		(net "/5V")
-	)
-	(segment
 		(start 171.601574 88.1)
 		(end 172.4 88.1)
@@
 	)
 	(segment
-		(start 147.4 84.7)
-		(end 153.65408 84.7)
-		(width 0.5)
-		(layer "F.Cu")
-		(net "/5V")
-	)
-	(segment
-		(start 172.4 85.5)
-		(end 172.4 88.732374)
+		(start 136.325 100.1)
+		(end 136.325 101.085)
 		(width 0.5)
 		(layer "F.Cu")
@@
 	)
 	(segment
-		(start 171.319107 103.380893)
-		(end 170.801574 103.380893)
+		(start 144.623574 90.25)
+		(end 144.773574 90.4)
 		(width 0.5)
 		(layer "F.Cu")
@@
 	)
 	(segment
-		(start 136.325 100.1)
-		(end 136.325 101.085)
+		(start 171.561574 100)
+		(end 171.561574 103.138426)
 		(width 0.5)
 		(layer "F.Cu")
@@
 	)
 	(segment
-		(start 169.4 91.732374)
-		(end 169.4 99.875001)
+		(start 135.717533 100.1)
+		(end 136.325 100.1)
 		(width 0.5)
 		(layer "F.Cu")
@@
 	)
 	(segment
-		(start 169.524999 100)
-		(end 170.2 100)
+		(start 153.95408 85)
+		(end 171.9 85)
 		(width 0.5)
 		(layer "F.Cu")
@@
 	)
 	(segment
-		(start 144.623574 90.25)
-		(end 144.773574 90.4)
+		(start 144.6 87.6625)
+		(end 144.773574 87.836074)
 		(width 0.5)
 		(layer "F.Cu")
@@
 	)
 	(segment
-		(start 135.717533 100.1)
-		(end 136.325 100.1)
-		(width 0.5)
-		(layer "F.Cu")
-		(net "/5V")
-	)
-	(segment
-		(start 144.6 87.6625)
-		(end 144.773574 87.836074)
+		(start 172.8 100)
+		(end 169.524999 100)
 		(width 0.5)
 		(layer "F.Cu")
@@
 	)
 	(segment
+		(start 146.8 85.3)
+		(end 147.4 84.7)
+		(width 0.5)
+		(layer "F.Cu")
+		(net "/5V")
+	)
+	(segment
 		(start 144.773574 90.4)
 		(end 144.773574 93.261426)
@@
 	)
 	(segment
-		(start 172.4 88.732374)
-		(end 169.4 91.732374)
-		(width 0.5)
-		(layer "F.Cu")
-		(net "/5V")
-	)
-	(segment
 		(start 136.64 103.4)
 		(end 136.65 103.39)
@@
 	)
 	(segment
-		(start 167.06 78.562846)
-		(end 164.901953 80.720893)
+		(start 164.901953 80.720893)
+		(end 163.101574 80.720893)
 		(width 0.635)
 		(layer "F.Cu")
@@
 	)
 	(segment
-		(start 167.06 76.24)
-		(end 167.06 78.562846)
+		(start 166.91 76.36)
+		(end 166.91 78.712846)
 		(width 0.635)
 		(layer "F.Cu")
@@
 	)
 	(segment
-		(start 164.901953 80.720893)
-		(end 163.101574 80.720893)
+		(start 166.91 78.712846)
+		(end 164.901953 80.720893)
 		(width 0.635)
 		(layer "F.Cu")

Commit message: diecast-2x2: user layout edits (KiCad save)
Parts:
- removed R2: 0R, Resistor_SMD:R_0805_2012Metric
- removed R26: NP, Resistor_SMD:R_0805_2012Metric
- removed U7: ADP150AUJZ-3.3-R7, Package_TO_SOT_SMD:SOT-23-5
- added C34: 10n, Synthesizer:Cap_0402, F.Cu at (213.8, 81.9)
- added C35: 1u 10V, Synthesizer:Cap_0402, F.Cu at (172.8, 100.2)
- added C39: 1u 10V, Synthesizer:Cap_0402, F.Cu at (167.5, 100.2)
- added C50: 100n, Synthesizer:Cap_0402, F.Cu at (216.7, 85.9)
- added C51: 100n, Synthesizer:Cap_0402, F.Cu at (219.5, 74.1)
- added C52: 1u 10V, Synthesizer:Cap_0402, F.Cu at (172.8, 104.4)
- added C53: 1u 10V, Synthesizer:Cap_0402, F.Cu at (167.6, 104.4)
- added D10: B5819W, Diode_SMD:D_SOD-123, F.Cu at (136.2, 110.6)
- added D9: B5819W, Diode_SMD:D_SOD-123, F.Cu at (171.5, 93.0)
- added J10: REF_OUT, Connector_Coaxial:SMA_Amphenol_901-144_Vertical, F.Cu at (151.9, 76.4)
- added J11: Header 1x3, Connector_PinHeader_2.54mm:PinHeader_1x03_P2.54mm_Vertical, F.Cu at (153.5, 88.8)
- added R28: 1M, Synthesizer:Res_0402, F.Cu at (222.4, 76.0)
- added R29: 47R, Synthesizer:Res_0402, F.Cu at (222.4, 78.0)
- added R30: 220R, Synthesizer:Res_0402, F.Cu at (222.4, 80.0)
- added R31: 510R, Synthesizer:Res_0402, F.Cu at (222.4, 81.9)
- added R32: 47R, Synthesizer:Res_0402, F.Cu at (222.4, 83.9)
- added U10: LP5907MFX-3.3, Package_TO_SOT_SMD:SOT-23-5, F.Cu at (170.1, 96.0)
- added U11: SN74LVC1GU04DBVR, Package_TO_SOT_SMD:SOT-23-5, F.Cu at (151.4, 82.8)
- added U6: LP5907MFX-3.3, Package_TO_SOT_SMD:SOT-23-5, F.Cu at (170.1, 99.8)
- added U9: LP5907MFX-3.3, Package_TO_SOT_SMD:SOT-23-5, F.Cu at (170.2, 103.9)
- J5: moved to F.Cu
- U8: value ADP150AUJZ-3.3-R7 -> LP5907MFX-3.3
- moved C41 66.2 mm to (134.8, 81.3)
- moved C40 65.1 mm to (136.6, 84.0)
- moved C5 62.5 mm to (213.8, 76.0), turned to 0 degrees
- moved R7 60.6 mm to (222.4, 74.1), turned to 0 degrees
- moved C42 59.6 mm to (141.7, 85.0)
- moved R6 58.2 mm to (219.5, 85.9), turned to 0 degrees
- moved C43 57.4 mm to (143.9, 86.6)
- moved R5 57.0 mm to (219.5, 83.9), turned to 0 degrees
- moved C4 51.2 mm to (213.8, 74.1), turned to 0 degrees
- moved L1 40.6 mm to (142.2, 82.3)
- moved C1 32.3 mm to (116.1, 93.0)
- moved D1 32.3 mm to (116.1, 91.2)
- moved J1 29.5 mm to (119.5, 119.8)
- moved U1 21.5 mm to (117.4, 108.9)
- moved C27 8.97 mm to (167.4, 96.6)
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Connections:
- net /VCC_2 renamed /VRF
- net Net-(R26-Pad2) renamed /REF_IN
- C13 pad 1: /VCC_1 -> /VDIG
- C18 pad 1: /VCC_1 -> /VVCO
- C19 pad 2: /VCC_1 -> /VDIG
- C21 pad 2: /VCC_1 -> /VDIG
- C24 pad 1: /VCC_1 -> /VADD
- C25 pad 1: /VCC_1 -> /VADD
- C27 pad 1: /VCC_1 -> /VDIG
- C28 pad 2: /VCC_1 -> /VVCO
- C29 pad 1: /5V -> /VDD
- C30 pad 1: /VCC_1 -> /VDIG
- C42 pad 1: /5V -> /5V_USB
- C43 pad 1: /5V -> /5V_USB
- C6 pad 1: /5V -> /5V_REG
- C8 pad 1: /5V -> /5V_REG
- D8 pad 2: Net-(D8-A) -> unconnected-(D8-A-Pad2)
- FB1 pad 2: /5V -> /5V_USB
- U1 pad 3: /5V -> /5V_REG
- U3 pad 2: Net-(D8-A) -> unconnected-(U3-PA3-Pad2)
- U3 pad 4: /5V -> /VDD
- U4 pad 10: /VCC_1 -> /VADD
- U4 pad 16: /VCC_1 -> /VVCO
- U4 pad 17: /VCC_1 -> /VVCO
- U4 pad 28: /VCC_1 -> /VDIG
- U4 pad 32: /VCC_1 -> /VDIG
- U4 pad 6: /VCC_1 -> /VADD
Routing:
- net /5V: track 100.1 -> 48.7 mm
- net /VCC_1: track 20.8 -> 0.00 mm, vias 8 -> 0
- net GND: track 58.4 -> 45.6 mm, vias 201 -> 169
- net /MUX: track 29.3 -> 16.6 mm, vias 4 -> 2
- net /LD: track 26.8 -> 15.9 mm, vias 2 -> 0
- net Net-(U4-REFIN): track 10.5 -> 2.08 mm, vias 2 -> 1
- net /VDIG: track 0.00 -> 7.52 mm, vias 0 -> 2
- net /VVCO: track 0.00 -> 5.61 mm, vias 0 -> 2
- net /VRF: track 15.1 -> 11.2 mm
- net /REF_IN: track 3.92 -> 0.00 mm
- net /VADD: track 0.00 -> 3.33 mm, vias 0 -> 2
- net (no net): track 0.00 -> 2.96 mm
- net Net-(J9-In): track 12.3 -> 9.49 mm
- net Net-(D8-A): track 2.66 -> 0.00 mm
- net /5V_REG: track 0.00 -> 2.42 mm
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
Commit message: prelim edits while working with grok
Parts:
- removed C1: 330n 50V, Capacitor_SMD:C_0603_1608Metric
- removed C16, C6: 100n, Synthesizer:Cap_0402
- removed C26, C37: 10p, Synthesizer:Cap_0402
- removed C27, C32, C52, C53: 1u 10V, Synthesizer:Cap_0402
- removed C8: 6.8u, Capacitor_SMD:C_0603_1608Metric
- removed D1: D_Schottky, Diode_SMD:D_0603_1608Metric
- removed D10: B5819W, Diode_SMD:D_SOD-123
- removed D4, D5: Yellow, LED_SMD:LED_0402_1005Metric
- removed D7: PA2, LED_SMD:LED_0402_1005Metric
- removed D8: PA3, LED_SMD:LED_0402_1005Metric
- removed J1: Screw_Terminal_01x02, TerminalBlock_TE-Connectivity:TerminalBlock_TE_282834-2_1x02_P2.54mm_Horizontal
- removed J11, J8: Header 1x3, Connector_PinHeader_2.54mm:PinHeader_1x03_P2.54mm_Vertical
- removed J6: Scope, Connector_PinHeader_2.54mm:PinHeader_1x03_P2.54mm_Vertical
- removed R10, R12, R17, R19, R8: 1K, Synthesizer:Res_0402
- removed R31: 510R, Synthesizer:Res_0402
- removed R32: 47R, Synthesizer:Res_0402
- removed R5: 49R9, Synthesizer:Res_0402
- removed R6: 330R, Synthesizer:Res_0402
- removed R7: 15R, Synthesizer:Res_0402
- removed U1: LM7805A, Package_TO_SOT_SMD:TO-252-2
- removed U10, U9: LP5907MFX-3.3, Package_TO_SOT_SMD:SOT-23-5
- added C54: 100n, Synthesizer:Cap_0402, F.Cu at (201.9, 88.5)
- added C55: 150p, Capacitor_SMD:C_0603_1608Metric, F.Cu at (202.5, 103.1)
- added C56: 2.2n, Capacitor_SMD:C_0603_1608Metric, F.Cu at (202.5, 105.6)
- added C57: 100n, Synthesizer:Cap_0402, F.Cu at (201.9, 90.4)
- added C58: 100n, Synthesizer:Cap_0402, F.Cu at (201.9, 92.4)
- added C59: 100p, Synthesizer:Cap_0402, F.Cu at (201.9, 94.4)
- added C60: 100n, Synthesizer:Cap_0402, F.Cu at (201.9, 96.3)
- added C61: 100n, Synthesizer:Cap_0402, F.Cu at (201.9, 98.3)
- added C62: 100n, Synthesizer:Cap_0402, F.Cu at (204.8, 86.5)
- added C63: 100n, Synthesizer:Cap_0402, F.Cu at (204.8, 88.5)
- added C65: 100n, Synthesizer:Cap_0402, F.Cu at (204.8, 90.4)
- added D11: PWR, Synthesizer:LED_KPTL-3216_ReverseMount, F.Cu at (216.4, 87.2)
- added D12: REF LOCK, Synthesizer:LED_KPTL-3216_ReverseMount, F.Cu at (216.4, 90.5)
- added D13: SYNTH LOCK, Synthesizer:LED_KPTL-3216_ReverseMount, F.Cu at (216.4, 93.9)
- added D14: COMM, Synthesizer:LED_KPTL-3216_ReverseMount, F.Cu at (216.4, 97.2)
- added FB2: BLM18KG601SN1D, Inductor_SMD:L_0603_1608Metric, F.Cu at (202.5, 108.1)
- added J12: UPDI, Synthesizer:TestPad_1x03_P2.54mm, F.Cu at (219.5, 102.2)
- added R33: 10k, Synthesizer:Res_0402, F.Cu at (204.8, 94.4)
- added R34: 10M, Resistor_SMD:R_0603_1608Metric, F.Cu at (202.5, 110.6)
- added R35: 5K1, Synthesizer:Res_0402, F.Cu at (204.8, 96.3)
- added R36: 100k, Synthesizer:Res_0402, F.Cu at (204.8, 98.3)
- added R37: 1k, Synthesizer:Res_0402, F.Cu at (207.7, 86.5)
- added R38: 1k, Synthesizer:Res_0402, F.Cu at (207.7, 88.5)
- added R39: 1k, Synthesizer:Res_0402, F.Cu at (207.7, 90.4)
- added R40: 1k, Synthesizer:Res_0402, F.Cu at (207.7, 92.4)
- added R41: 51R, Resistor_SMD:R_0603_1608Metric, F.Cu at (206.5, 100.5)
- added R44: 33R, Synthesizer:Res_0402, F.Cu at (207.7, 94.4)
- added R46: 10k, Resistor_SMD:R_0603_1608Metric, F.Cu at (206.5, 103.1)
- added R47: 10k, Resistor_SMD:R_0603_1608Metric, F.Cu at (206.5, 105.6)
- added R48: 100k, Resistor_SMD:R_0603_1608Metric, F.Cu at (206.5, 108.1)
- added R49: 100k, Resistor_SMD:R_0603_1608Metric, F.Cu at (206.5, 110.6)
- added U12: ADF4002BCPZ, Package_DFN_QFN:QFN-20-1EP_4x4mm_P0.5mm_EP2.5x2.5mm, F.Cu at (182.5, 86.1)
- added U13: SN74LVC1GU04DBVR, Package_TO_SOT_SMD:SOT-23-5, F.Cu at (217.9, 106.5)
- C12, C23: value 100p -> 1n
- C17: value 4.7n -> 3.3n
- C20: value 2.7n -> 100p
- C31: value 680p -> 150p
- C34: value 10n -> 100p
- C4, C5: value 10n -> 100n
- J2: footprint Connector_PinHeader_2.54mm:PinHeader_1x03_P2.54mm_Vertical -> Connector_PinHeader_2.54mm:PinHeader_1x05_P2.54mm_Vertical
- J4: moved to F.Cu
- R14: value 560R -> 2.2K
- R25: value 1K -> 2.7K
- R29: value 47R -> 39R
- R30: value 220R -> 1M
- X1: value HCI 8122S-25NQ33FTL -> IQXT-220-2 10MHz; footprint Synthesizer:Oscillator_SMD2520 -> Synthesizer:Oscillator_SMD_3225_VCTCXO
- moved J2 47.1 mm to (211.4, 87.8), turned to 0 degrees
- moved U5 25.5 mm to (137.9, 82.0)
- moved X1 24.5 mm to (171.1, 86.8)
- moved R30 21.5 mm to (204.8, 92.4)
- moved U11 15.0 mm to (165.9, 87.0)
- moved C34 12.7 mm to (201.9, 86.5)
- moved C41 3.78 mm to (134.0, 85.0)
- moved J4 1.30 mm to (142.3, 75.1), turned to 180 degrees
- moved C40 1.05 mm to (136.6, 85.0)
- moved L1 0.90 mm to (143.0, 82.0), turned to -90 degrees
Connections:
- net Net-(X1-OUT) renamed /XO
- C13 pad 1: /VDIG -> /VDD
- C19 pad 2: /VDIG -> /VDD
- C21 pad 2: /VDIG -> /VDD
- C24 pad 1: /VADD -> /VRF
- C25 pad 1: /VADD -> /VRF
- C3 pad 2: Net-(C3-Pad2) -> /BUF
- C30 pad 1: /VDIG -> /VDD
- C34 pad 1: Net-(C34-Pad1) -> GND
- C5 pad 2: /VCC_1 -> /VDD
- C51 pad 2: /VCC_1 -> /VDD
- J2 pad 3: GND -> /DBG1
- L1 pad 1: Net-(L1-Pad1) -> Net-(J4-D--PadA7)
- L1 pad 2: Net-(L1-Pad2) -> Net-(J4-D+-PadA6)
- L1 pad 3: /USB_DP -> Net-(L1-Pad3)
- L1 pad 4: /USB_DM -> Net-(L1-Pad4)
- R28 pad 2: Net-(R28-Pad2) -> /BUF
- R29 pad 1: Net-(C34-Pad1) -> /REF_OUT
- R29 pad 2: Net-(R28-Pad2) -> /BUF
- R30 pad 1: Net-(R28-Pad2) -> Net-(C4-Pad1)
- U11 pad 4: Net-(R28-Pad2) -> /BUF
- U11 pad 5: /VCC_1 -> /VDD
- U2 pad 1: /RXD_U -> /TXD_M
- U2 pad 14: /RXLED/ -> unconnected-(U2-CBUS1-Pad14)
- U2 pad 18: unconnected-(U2-~{DTR}-Pad18) -> /DTR
- U2 pad 20: /3V3 -> /VDD
- U2 pad 7: /TXLED/ -> /CBUS_ACT
- U3 pad 1: Net-(D7-A) -> unconnected-(U3-PA2-Pad1)
- U3 pad 10: Net-(J6-Pin_3) -> /REF_LOCK
- U3 pad 5: unconnected-(U3-PA4-Pad5) -> /RST
- U3 pad 6: unconnected-(U3-PA5-Pad6) -> /MUX4002
- U3 pad 7: unconnected-(U3-PA6-Pad7) -> /DAC_HOLD
- U3 pad 8: unconnected-(U3-PA7-Pad8) -> /LE4002
- U3 pad 9: Net-(J6-Pin_2) -> /SYNTH_LOCK
- U4 pad 10: /VADD -> /VRF
- U4 pad 19: Net-(U4-TEMP) -> unconnected-(U4-TEMP-Pad19)
- U4 pad 28: /VDIG -> /VDD
- U4 pad 32: /VDIG -> /VDD
- U4 pad 6: /VADD -> /VRF
- U5 pad 1: Net-(J4-D--PadA7) -> Net-(L1-Pad4)
- U5 pad 3: Net-(J4-D+-PadA6) -> Net-(L1-Pad3)
- U5 pad 4: Net-(L1-Pad2) -> /USB_DP
- U5 pad 6: Net-(L1-Pad1) -> /USB_DM
- X1 pad 1: GND -> /CP
- X1 pad 4: /VCC_1 -> /VDD
Routing:
- net (no net): track 2.96 -> 18.6 mm, vias 0 -> 1
- net /VDIG: track 7.52 -> 0.00 mm, vias 2 -> 0
- net /VDD: track 0.00 -> 7.52 mm, vias 0 -> 2
- net /12V: track 6.52 -> 0.00 mm
- net Net-(J6-Pin_3): track 5.68 -> 0.00 mm
- net /REF_LOCK: track 0.00 -> 5.68 mm
- net Net-(J6-Pin_2): track 4.50 -> 0.00 mm
- net /SYNTH_LOCK: track 0.00 -> 4.50 mm
- net /RXD_U: track 4.44 -> 0.00 mm, vias 1 -> 0
- net /TXD_M: track 15.7 -> 20.1 mm, vias 0 -> 1
- net unconnected-(U3-PA2-Pad1): track 0.00 -> 4.19 mm
- net Net-(D7-A): track 4.19 -> 0.00 mm
- net Net-(D1-K): track 4.01 -> 0.00 mm
- net unconnected-(U2-CBUS1-Pad14): track 0.00 -> 3.54 mm, vias 0 -> 2
- net /RXLED/: track 3.54 -> 0.00 mm, vias 2 -> 0
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- added copper zone on In2.Cu, net /VDD
- removed copper zone on In2.Cu, net /VCC_1
